Commit message: all bots

File: bullet3/data/bipedal2.urdf (robot description, URDF)
Before this commit: robot bipedal, 11 links, 10 joints
Links:
- removed link left_leg_cube
- removed link left_thigh_sphere
- removed link right_leg_cube
- removed link right_thigh_sphere
- link waist: geometry collision box size=0.16 0.60 .07; visual box size=0.16 0.60 .07
Joints:
- removed joint left_groin_joint
- removed joint left_groin_sphere
- removed joint left_knee_joint
- removed joint left_leg_cube_joint
- removed joint right_groin_joint
- removed joint right_groin_sphere
- removed joint right_knee_joint
- removed joint right_leg_cube_joint
- added joint left_groin: type continuous, parent waist, child left_thigh, origin xyz=0 -0.22 -0.35 rpy=0 0 0, axis 0 1 0, limit effort=100 velocity=100
- added joint left_knee: type continuous, parent left_thigh, child left_leg, origin xyz=0 0 -0.565 rpy=0 0 0, axis 0 1 0, limit effort=100 velocity=100
- added joint right_groin: type continuous, parent waist, child right_thigh, origin xyz=0 0.22 -0.35 rpy=0 0 0, axis 0 1 0, limit effort=100 velocity=100
- added joint right_knee: type continuous, parent right_thigh, child right_leg, origin xyz=0 0 -0.565 rpy=0 0 0, axis 0 1 0, limit effort=100 velocity=100

File: bullet3/data/cheetah.urdf (robot description, URDF)
Before this commit: robot spider, 26 links, 25 joints
Links:
- link back_left_1: mass 0.06 -> 0.25
- link back_left_2: mass 0.06 -> 0.25
- link back_left_3: mass 0.015 -> 0.25
- link back_left_4: mass 0.06 -> 0.25
- link back_left_5: mass 0.015 -> 0.25
- link back_left_6: mass 0.015 -> 0.25
- link back_right_1: mass 0.06 -> 0.25
- link back_right_2: mass 0.06 -> 0.25
- link back_right_3: mass 0.015 -> 0.25
- link back_right_4: mass 0.06 -> 0.25
- link back_right_5: mass 0.015 -> 0.25
- link back_right_6: mass 0.015 -> 0.25
- link base_chassis_link: mass 0.2 -> 10; geometry collision box size=0.80 0.30 0.20; visual box size=0.80 0.30 0.20
- link front_left_1: mass 0.06 -> 0.25
- link front_left_2: mass 0.06 -> 0.25
- link front_left_3: mass 0.015 -> 0.25
- link front_left_4: mass 0.06 -> 0.25
- link front_left_5: mass 0.015 -> 0.25
- link front_left_6: mass 0.015 -> 0.25
- link front_right_1: mass 0.06 -> 0.25
- link front_right_2: mass 0.06 -> 0.25
- link front_right_3: mass 0.015 -> 0.25
- link front_right_4: mass 0.06 -> 0.25
- link front_right_5: mass 0.015 -> 0.25
- link front_right_6: mass 0.015 -> 0.25
- link head: mass 0.06 -> 0.5
